Commit message: Add functional structure

File: urdf/gpg.urdf (robot description, URDF)
Before this commit: robot myrobot, 4 links, 3 joints
Links:
- added link base_footprint; visual box size=0.05 0.05 0.001
Joints:
- added joint base_joint: type fixed, parent base_footprint, child base_link, origin xyz=0 0 0.03 rpy=0 0 0
- joint left_wheel: axis (none) -> 0 1 0
- joint right_wheel: axis (none) -> 0 1 0
- joint servo: axis (none) -> 0 0 1; limit (none) -> lower=-0.12 upper=0.12 effort=1000.0 velocity=0.5; type fixed -> revolute
